Commit message: feat: Add new features and update environment for bimanual manipulation

File: env_setup/robot_setting/openarm_tesollo_t3.urdf (robot description, URDF)
Before this commit: robot openarm_tesollo_mount, 113 links, 112 joints
Links:
- removed link tesollo_left_finger_1_seg1_sensor_link
- removed link tesollo_left_finger_1_seg2_sensor_link
- removed link tesollo_left_finger_1_seg4_sensor_link
- removed link tesollo_left_finger_2_seg1_sensor_link
- removed link tesollo_left_finger_2_seg4_sensor_link
- removed link tesollo_left_finger_3_seg1_sensor_link
- removed link tesollo_left_finger_3_seg4_sensor_link
- removed link tesollo_left_finger_4_seg1_sensor_link
- removed link tesollo_left_finger_4_seg4_sensor_link
- removed link tesollo_left_finger_5_seg1_sensor_link
- removed link tesollo_left_finger_5_seg2_sensor_link
- removed link tesollo_left_finger_5_seg4_sensor_link
- removed link tesollo_left_palm_sensor_link
- removed link tesollo_right_finger_1_seg1_sensor_link
- removed link tesollo_right_finger_1_seg2_sensor_link
- removed link tesollo_right_finger_1_seg4_sensor_link
- removed link tesollo_right_finger_2_seg1_sensor_link
- removed link tesollo_right_finger_2_seg4_sensor_link
- removed link tesollo_right_finger_3_seg1_sensor_link
- removed link tesollo_right_finger_3_seg4_sensor_link
- removed link tesollo_right_finger_4_seg1_sensor_link
- removed link tesollo_right_finger_4_seg4_sensor_link
- removed link tesollo_right_finger_5_seg1_sensor_link
- removed link tesollo_right_finger_5_seg2_sensor_link
- removed link tesollo_right_finger_5_seg4_sensor_link
- removed link tesollo_right_palm_sensor_link
- added link tesollo_left_palm_sensor_link1, mass 0.001; collision cylinder length=0.001 radius=0.005; visual cylinder length=0.001 radius=0.005
- added link tesollo_left_palm_sensor_link2, mass 0.001; collision cylinder length=0.001 radius=0.005; visual cylinder length=0.001 radius=0.005
- added link tesollo_left_palm_sensor_link3, mass 0.001; collision cylinder length=0.001 radius=0.005; visual cylinder length=0.001 radius=0.005
- added link tesollo_right_palm_sensor_link1, mass 0.001; collision cylinder length=0.001 radius=0.005; visual cylinder length=0.001 radius=0.005
- added link tesollo_right_palm_sensor_link2, mass 0.001; collision cylinder length=0.001 radius=0.005; visual cylinder length=0.001 radius=0.005
- added link tesollo_right_palm_sensor_link3, mass 0.001; collision cylinder length=0.001 radius=0.005; visual cylinder length=0.001 radius=0.005
- link tesollo_left_finger_1_seg3_sensor_link: mass None -> 0.001; geometry collision cylinder length=0.001 radius=0.005; visual cylinder length=0.001 radius=0.005
- link tesollo_left_finger_1_tip_sensor_link: mass None -> 0.001; geometry collision cylinder length=0.001 radius=0.005; visual cylinder length=0.001 radius=0.005
- link tesollo_left_finger_2_seg2_sensor_link: mass None -> 0.001; geometry collision cylinder length=0.001 radius=0.005; visual cylinder length=0.001 radius=0.005
- link tesollo_left_finger_2_seg3_sensor_link: mass None -> 0.001; geometry collision cylinder length=0.001 radius=0.005; visual cylinder length=0.001 radius=0.005
- link tesollo_left_finger_2_tip_sensor_link: mass None -> 0.001; geometry collision cylinder length=0.001 radius=0.005; visual cylinder length=0.001 radius=0.005
- link tesollo_left_finger_3_seg2_sensor_link: mass None -> 0.001; geometry collision cylinder length=0.001 radius=0.005; visual cylinder length=0.001 radius=0.005
- link tesollo_left_finger_3_seg3_sensor_link: mass None -> 0.001; geometry collision cylinder length=0.001 radius=0.005; visual cylinder length=0.001 radius=0.005
- link tesollo_left_finger_3_tip_sensor_link: mass None -> 0.001; geometry collision cylinder length=0.001 radius=0.005; visual cylinder length=0.001 radius=0.005
- link tesollo_left_finger_4_seg2_sensor_link: mass None -> 0.001; geometry collision cylinder length=0.001 radius=0.005; visual cylinder length=0.001 radius=0.005
- link tesollo_left_finger_4_seg3_sensor_link: mass None -> 0.001; geometry collision cylinder length=0.001 radius=0.005; visual cylinder length=0.001 radius=0.005
- link tesollo_left_finger_4_tip_sensor_link: mass None -> 0.001; geometry collision cylinder length=0.001 radius=0.005; visual cylinder length=0.001 radius=0.005
- link tesollo_left_finger_5_seg3_sensor_link: mass None -> 0.001; geometry collision cylinder length=0.001 radius=0.005; visual cylinder length=0.001 radius=0.005
- link tesollo_left_finger_5_tip_sensor_link: mass None -> 0.001; geometry collision cylinder length=0.001 radius=0.005; visual cylinder length=0.001 radius=0.005
- link tesollo_right_finger_1_seg3_sensor_link: mass None -> 0.001; geometry collision cylinder length=0.001 radius=0.005; visual cylinder length=0.001 radius=0.005
- link tesollo_right_finger_1_tip_sensor_link: mass None -> 0.001; geometry collision cylinder length=0.001 radius=0.005; visual cylinder length=0.001 radius=0.005
- link tesollo_right_finger_2_seg2_sensor_link: mass None -> 0.001; geometry collision cylinder length=0.001 radius=0.005; visual cylinder length=0.001 radius=0.005
- link tesollo_right_finger_2_seg3_sensor_link: mass None -> 0.001; geometry collision cylinder length=0.001 radius=0.005; visual cylinder length=0.001 radius=0.005
- link tesollo_right_finger_2_tip_sensor_link: mass None -> 0.001; geometry collision cylinder length=0.001 radius=0.005; visual cylinder length=0.001 radius=0.005
- link tesollo_right_finger_3_seg2_sensor_link: mass None -> 0.001; geometry collision cylinder length=0.001 radius=0.005; visual cylinder length=0.001 radius=0.005
- link tesollo_right_finger_3_seg3_sensor_link: mass None -> 0.001; geometry collision cylinder length=0.001 radius=0.005; visual cylinder length=0.001 radius=0.005
- link tesollo_right_finger_3_tip_sensor_link: mass None -> 0.001; geometry collision cylinder length=0.001 radius=0.005; visual cylinder length=0.001 radius=0.005
- link tesollo_right_finger_4_seg2_sensor_link: mass None -> 0.001; geometry collision cylinder length=0.001 radius=0.005; visual cylinder length=0.001 radius=0.005
- link tesollo_right_finger_4_seg3_sensor_link: mass None -> 0.001; geometry collision cylinder length=0.001 radius=0.005; visual cylinder length=0.001 radius=0.005
- link tesollo_right_finger_4_tip_sensor_link: mass None -> 0.001; geometry collision cylinder length=0.001 radius=0.005; visual cylinder length=0.001 radius=0.005
- link tesollo_right_finger_5_seg3_sensor_link: mass None -> 0.001; geometry collision cylinder length=0.001 radius=0.005; visual cylinder length=0.001 radius=0.005
- link tesollo_right_finger_5_tip_sensor_link: mass None -> 0.001; geometry collision cylinder length=0.001 radius=0.005; visual cylinder length=0.001 radius=0.005
Joints:
- removed joint tesollo_left_finger_1_seg1_sensor_joint
- removed joint tesollo_left_finger_1_seg2_sensor_joint
- removed joint tesollo_left_finger_1_seg4_sensor_joint
- removed joint tesollo_left_finger_2_seg1_sensor_joint
- removed joint tesollo_left_finger_2_seg4_sensor_joint
- removed joint tesollo_left_finger_3_seg1_sensor_joint
- removed joint tesollo_left_finger_3_seg4_sensor_joint
- removed joint tesollo_left_finger_4_seg1_sensor_joint
- removed joint tesollo_left_finger_4_seg4_sensor_joint
- removed joint tesollo_left_finger_5_seg1_sensor_joint
- removed joint tesollo_left_finger_5_seg2_sensor_joint
- removed joint tesollo_left_finger_5_seg4_sensor_joint
- removed joint tesollo_left_palm_sensor_joint
- removed joint tesollo_right_finger_1_seg1_sensor_joint
- removed joint tesollo_right_finger_1_seg2_sensor_joint
- removed joint tesollo_right_finger_1_seg4_sensor_joint
- removed joint tesollo_right_finger_2_seg1_sensor_joint
- removed joint tesollo_right_finger_2_seg4_sensor_joint
- removed joint tesollo_right_finger_3_seg1_sensor_joint
- removed joint tesollo_right_finger_3_seg4_sensor_joint
- removed joint tesollo_right_finger_4_seg1_sensor_joint
- removed joint tesollo_right_finger_4_seg4_sensor_joint
- removed joint tesollo_right_finger_5_seg1_sensor_joint
- removed joint tesollo_right_finger_5_seg2_sensor_joint
- removed joint tesollo_right_finger_5_seg4_sensor_joint
- removed joint tesollo_right_palm_sensor_joint
- added joint tesollo_left_palm_sensor_joint1: type fixed, parent tesollo_left_ll_dg_mount, child tesollo_left_palm_sensor_link1, origin xyz=0.02 -0.02 0.14 rpy=0 1.5708 0
- added joint tesollo_left_palm_sensor_joint2: type fixed, parent tesollo_left_ll_dg_mount, child tesollo_left_palm_sensor_link2, origin xyz=0.02 0.0 0.14 rpy=0 1.5708 0
- added joint tesollo_left_palm_sensor_joint3: type fixed, parent tesollo_left_ll_dg_mount, child tesollo_left_palm_sensor_link3, origin xyz=0.02 0.02 0.14 rpy=0 1.5708 0
- added joint tesollo_right_palm_sensor_joint1: type fixed, parent tesollo_right_rl_dg_mount, child tesollo_right_palm_sensor_link1, origin xyz=0.02 -0.02 0.14 rpy=0 1.5708 0
- added joint tesollo_right_palm_sensor_joint2: type fixed, parent tesollo_right_rl_dg_mount, child tesollo_right_palm_sensor_link2, origin xyz=0.02 0 0.14 rpy=0 1.5708 0
- added joint tesollo_right_palm_sensor_joint3: type fixed, parent tesollo_right_rl_dg_mount, child tesollo_right_palm_sensor_link3, origin xyz=0.02 0.02 0.14 rpy=0 1.5708 0
- joint tesollo_left_finger_1_seg3_sensor_joint: origin xyz=0 0 0.001 rpy=0 0 0 -> xyz=0 -0.015 0.0095 rpy=0 0 0
- joint tesollo_left_finger_1_tip_sensor_joint: origin xyz=0 -0.001 0 rpy=0 0 0 -> xyz=0 -0.045 0.01 rpy=0.261799 0 0
- joint tesollo_left_finger_2_seg2_sensor_joint: origin xyz=0 0 0.001 rpy=0 0 0 -> xyz=0.0095 0 0.02 rpy=0 1.5708 0
- joint tesollo_left_finger_2_seg3_sensor_joint: origin xyz=0 0 0.001 rpy=0 0 0 -> xyz=0.0095 0 0.02 rpy=0 1.5708 0
- joint tesollo_left_finger_2_tip_sensor_joint: origin xyz=0 0 0.001 rpy=0 0 0 -> xyz=0.01 0 0.035 rpy=0 1.3089969389957472 0
- joint tesollo_left_finger_3_seg2_sensor_joint: origin xyz=0 0 0.001 rpy=0 0 0 -> xyz=0.0095 0 0.02 rpy=0 1.5708 0
- joint tesollo_left_finger_3_seg3_sensor_joint: origin xyz=0 0 0.001 rpy=0 0 0 -> xyz=0.0095 0 0.02 rpy=0 1.5708 0
- joint tesollo_left_finger_3_tip_sensor_joint: origin xyz=0 0 0.001 rpy=0 0 0 -> xyz=0.01 0 0.035 rpy=0 1.3089969389957472 0
- joint tesollo_left_finger_4_seg2_sensor_joint: origin xyz=0 0 0.001 rpy=0 0 0 -> xyz=0.0095 0 0.02 rpy=0 1.5708 0
- joint tesollo_left_finger_4_seg3_sensor_joint: origin xyz=0 0 0.001 rpy=0 0 0 -> xyz=0.0095 0 0.02 rpy=0 1.5708 0
- joint tesollo_left_finger_4_tip_sensor_joint: origin xyz=0 0 0.001 rpy=0 0 0 -> xyz=0.01 0 0.035 rpy=0 1.3089969389957472 0
- joint tesollo_left_finger_5_seg3_sensor_joint: origin xyz=0 0 0.001 rpy=0 0 0 -> xyz=0.0095 0 0.02 rpy=0 1.5708 0
- joint tesollo_left_finger_5_tip_sensor_joint: origin xyz=0 0 0.001 rpy=0 0 0 -> xyz=0.01 0 0.045 rpy=0 1.3089969389957472 0
- joint tesollo_right_finger_1_seg3_sensor_joint: origin xyz=0 0 0.001 rpy=0 0 0 -> xyz=0 0.015 0.0095 rpy=0 0 0
- joint tesollo_right_finger_1_tip_sensor_joint: origin xyz=0 0.001 0 rpy=0 0 0 -> xyz=0 0.045 0.01 rpy=-0.261799 0 0
- joint tesollo_right_finger_2_seg2_sensor_joint: origin xyz=0 0 0.001 rpy=0 0 0 -> xyz=0.0095 0 0.02 rpy=0 1.5708 0
- joint tesollo_right_finger_2_seg3_sensor_joint: origin xyz=0 0 0.001 rpy=0 0 0 -> xyz=0.0095 0 0.02 rpy=0 1.5708 0
- joint tesollo_right_finger_2_tip_sensor_joint: origin xyz=0 0 0.001 rpy=0 0 0 -> xyz=0.01 0 0.035 rpy=0 1.3089969389957472 0
- joint tesollo_right_finger_3_seg2_sensor_joint: origin xyz=0 0 0.001 rpy=0 0 0 -> xyz=0.0095 0 0.02 rpy=0 1.5708 0
- joint tesollo_right_finger_3_seg3_sensor_joint: origin xyz=0 0 0.001 rpy=0 0 0 -> xyz=0.0095 0 0.02 rpy=0 1.5708 0
- joint tesollo_right_finger_3_tip_sensor_joint: origin xyz=0 0 0.001 rpy=0 0 0 -> xyz=0.01 0 0.035 rpy=0 1.3089969389957472 0
- joint tesollo_right_finger_4_seg2_sensor_joint: origin xyz=0 0 0.001 rpy=0 0 0 -> xyz=0.0095 0 0.02 rpy=0 1.5708 0
- joint tesollo_right_finger_4_seg3_sensor_joint: origin xyz=0 0 0.001 rpy=0 0 0 -> xyz=0.0095 0 0.02 rpy=0 1.5708 0
- joint tesollo_right_finger_4_tip_sensor_joint: origin xyz=0 0 0.001 rpy=0 0 0 -> xyz=0.01 0 0.035 rpy=0 1.3089969389957472 0
- joint tesollo_right_finger_5_seg3_sensor_joint: origin xyz=0 0 0.001 rpy=0 0 0 -> xyz=0.0095 0 0.02 rpy=0 1.5708 0
- joint tesollo_right_finger_5_tip_sensor_joint: origin xyz=0 0 0.001 rpy=0 0 0 -> xyz=0.01 0 0.045 rpy=0 1.3089969389957472 0
